Commit message: axis orientation fix for copterlab gimbal

File: gimbal_urdf/urdf/gimbal_urdf.urdf (robot description, URDF)
Before this commit: robot gimbal_urdf, 5 links, 4 joints
Links:
- added link world
Joints:
- added joint base_joint: type fixed, parent world, child base_link, origin xyz=0.0 0.0 0.0 rpy=-0 0 3.14, limit lower=-3.14 upper=3.14 effort=30 velocity=1.0

Commit message: added 2 cam_links (left and right)

File: gimbal_urdf/urdf/gimbal_urdf.urdf (robot description, URDF)
Before this commit: robot gimbal_urdf, 6 links, 5 joints
Links:
- added link lcam_link, mass 0.0801973434031241; collision box size=0.02 0.02 0.02; visual box size=0.02 0.02 0.02
- added link rcam_link, mass 0.0801973434031241; collision box size=0.02 0.02 0.02; visual box size=0.02 0.02 0.02
Joints:
- added joint lcam_to_EE: type fixed, parent EE, child lcam_link, origin xyz=0.045 0 0 rpy=0 0 0, axis 0 0 0
- added joint rcam_to_EE: type fixed, parent EE, child rcam_link, origin xyz=-0.045 0 0 rpy=0 0 0, axis 0 0 0
